Commit message: Update simulation

File: smartfactory_ws/src/smartfactory/smartfactory_description/urdf/smart_spawn.urdf.xacro (robot description, xacro)
@@ -1,10 +1,3 @@
 <?xml version="1.0"?>
-<!--
-    - Base      : kobuki
-    - Stacks    : interbotix
-    - 3d Sensor : astra
-    - Lidar     : rplidar
-    - arm : TODO: supported arms?
--->
 <robot name="smart_cameras" xmlns:xacro="http://ros.org/wiki/xacro">
   <xacro:arg name="use_nominal_extrinsics" default="false" />

File: smartfactory_ws/src/turtlebot2i/turtlebot2i_description/urdf/common_properties.urdf.xacro (robot description, xacro)
@@ -8,4 +8,9 @@
     <material name="white">
       <color rgba="1 1 1 1"/>
+    </material>
+  </xacro:property>
+  <xacro:property name="material_near_black">
+    <material name="near_black">
+      <color rgba="0.125 0.125 0.125 1"/>
     </material>
   </xacro:property>

File: smartfactory_ws/src/turtlebot2i/turtlebot2i_description/urdf/stacks/sim_interbotix.urdf.xacro (robot description, xacro)
@@ -18,6 +18,6 @@
   <xacro:property name="STANDOFF_UTILITY_UPPER_Z" value="${PLATE_UTILITY_BOTTOM_Z+PLATE_HEIGHT/2.0+STANDOFF_100_HEIGHT/2.0}"/>
   <xacro:property name="PLATE_UTILITY_UPPER_Z" value="${STANDOFF_UTILITY_UPPER_Z+STANDOFF_100_HEIGHT/2.0+PLATE_HEIGHT/2.0}"/>
-  <xacro:property name="STANDOFF_TOP_Z" value="${PLATE_UTILITY_UPPER_Z+PLATE_HEIGHT/2.0+STANDOFF_100_HEIGHT/2.0}"/>
-  <xacro:property name="PLATE_TOP_Z" value="${STANDOFF_TOP_Z+STANDOFF_100_HEIGHT/2.0+PLATE_HEIGHT/2.0}"/>
+  <xacro:property name="STANDOFF_TOP_Z" value="${PLATE_UTILITY_UPPER_Z+PLATE_HEIGHT/2.0+STANDOFF_50_HEIGHT/2.0}"/>
+  <xacro:property name="PLATE_TOP_Z" value="${STANDOFF_TOP_Z+STANDOFF_50_HEIGHT/2.0+PLATE_HEIGHT/2.0}"/>
   <xacro:property name="STANDOFF_FRONT_Z" value="${PLATE_MIDDLE_Z+PLATE_HEIGHT/2.0+STANDOFF_258_HEIGHT/2.0}"/>
   <!-- Xacro macros -->
@@ -278,4 +278,40 @@
       <gravity>true</gravity>
     </gazebo>
+    <xacro:standoff_50mm parent="${parent}" number="12" x_loc= "-0.001" y_loc= "0.162" z_loc="${STANDOFF_TOP_Z}"/>
+    <xacro:standoff_50mm parent="${parent}" number="13" x_loc= "-0.001" y_loc="-0.162" z_loc="${STANDOFF_TOP_Z}"/>
+    <xacro:standoff_50mm parent="${parent}" number="14" x_loc="-0.104" y_loc= "0.098" z_loc="${STANDOFF_TOP_Z}"/>
+    <xacro:standoff_50mm parent="${parent}" number="15" x_loc="-0.104" y_loc="-0.098" z_loc="${STANDOFF_TOP_Z}"/>
+    <joint name="plate_top_joint" type="fixed">
+      <origin xyz="0.0 0.0 ${PLATE_TOP_Z}" rpy="0 0 0"/>
+      <parent link="${parent}"/>
+      <child link="plate_top_link"/>
+    </joint>
+    <link name="plate_top_link">
+      <visual>
+        <origin xyz="0 0 0" rpy="0 0 0"/>
+        <geometry>
+          <mesh filename="package://turtlebot2i_description/meshes/stacks/interbotix/TurtleBot2i_TopPlate.stl" scale="0.001 0.001 0.001"/>
+        </geometry>
+        <xacro:insert_block name="material_dark_grey"/>
+      </visual>
+      <collision>
+        <origin xyz="0 0 0" rpy="0 0 0"/>
+        <geometry>
+          <mesh filename="package://turtlebot2i_description/meshes/stacks/interbotix/TurtleBot2i_TopPlate.stl" scale="0.001 0.001 0.001"/>
+        </geometry>
+      </collision>
+      <inertial>
+        <mass value="0.377"/>
+        <origin xyz="0 0 0"/>
+        <inertia ixx="0.003328" ixy="0.0" ixz="0.0"
+                 iyy="0.003328" iyz="0.0"
+                 izz="0.006656" />
+      </inertial>
+    </link>
+    <gazebo reference="plate_top_link">
+      <material>Gazebo/DarkGrey</material>
+      <!-- <selfCollide>true</selfCollide> -->
+      <gravity>true</gravity>
+    </gazebo>
   </xacro:macro>
 </robot>
